File: 3d_printer_pcb/3d_printer_pcb.kicad_sch (KiCad schematic)
At the start: 1 part, among them U1 RaspberryPi-CM3+

Commit message: made references
Parts:
- removed U1: RaspberryPi-CM3+, symbol MCU_Module:RaspberryPi-CM3+
- added J1, J2: 10164228-1001A1RLF, 10164228-1001A1RLF:AMPHENOL_10164228-1001A1RLF, symbol 10164228-1001A1RLF:10164228-1001A1RLF

Commit message: iupdate to pcb made power
Parts:
- added PNLED1: power_on_led, LED_SMD:LED_1206_3216Metric_Pad1.42x1.75mm_HandSolder, symbol Device:LED
- added R1_led1: 270Ω, Resistor_THT:R_Axial_DIN0204_L3.6mm_D1.6mm_P5.08mm_Horizontal, symbol Device:R
- added R2_led2: 100Ω, Resistor_THT:R_Axial_DIN0204_L3.6mm_D1.6mm_P5.08mm_Horizontal, symbol Device:R
- added USBCLED1: usbc_led, LED_SMD:LED_1206_3216Metric_Pad1.42x1.75mm_HandSolder, symbol Device:LED
- added cmh1, cmh3, cmh4: cm5_hole, MountingHole:MountingHole_2.5mm_Pad, symbol Mechanical:MountingHole
- added cmh2: cm5_hole, symbol Mechanical:MountingHole
- added usbc1: usb_c_con_6p, symbol Connector:USB_C_Receptacle_PowerOnly_6P
- cmc1: renamed from J1; value 10164228-1001A1RLF -> cm5_10164228-1001A1RLF_c
- cmc2: renamed from J2; value 10164228-1001A1RLF -> cm5_10164228-1001A1RLF_c
Connections:
- net at cmc2.13: now also cmc1.1, cmc1.13, cmc1.14, cmc1.2, cmc1.22, cmc1.23, cmc1.32, cmc1.33, cmc1.42, cmc1.43, cmc1.52, cmc1.53, cmc1.59, cmc1.60, cmc1.65, cmc1.66, cmc1.7, cmc1.71, cmc1.74, cmc1.8, cmc2.14, cmc2.19, cmc2.20, cmc2.25, cmc2.26, cmc2.31, cmc2.32, cmc2.37, cmc2.38, cmc2.44, cmc2.50, cmc2.55, cmc2.56, cmc2.61, cmc2.62, cmc2.67, cmc2.68, cmc2.7, cmc2.73, cmc2.74, cmc2.79, cmc2.8, cmc2.80, cmc2.85, cmc2.86, cmc2.91, cmc2.92, cmc2.97, cmc2.98, usbc1.A12 (GND), usbc1.B12 (GND)
- net at cmc1.21: now also PNLED1.1 (K)
- net at cmc1.77: now also cmc1.79, cmc1.81, cmc1.83, cmc1.85, cmc1.87, R1_led1.2, usbc1.A9 (VBUS), usbc1.B9 (VBUS)
- net at cmc1.84: now also R2_led2.2
- net at cmc1.94: now also usbc1.A5 (CC1)
- net at cmc1.95: now also USBCLED1.1 (K)
- net at cmc1.96: now also usbc1.B5 (CC2)
- new net: R1_led1.1, USBCLED1.2 (A)
- new net: PNLED1.2 (A), R2_led2.1
Other:
- moved on the sheet: cmc1, cmc2
